File: src/linear/SCH and PCB/VupiterLinear Stage.kicad_pcb (KiCad board)
At the start: 2 copper layers, 68 parts, among them Q1 TIP41C, Q2 TIP41C, T1 2N3904, T2 2N3904

Commit message: Add files via upload
Parts:
- removed U$10, U$30, U$5: 3362P-1-502, BOCHEN_3362P-1-502
- removed U$24, U$25: LTR18, ROHM_LTR18
- removed U$26: ATS-PCBT1090, ATS_ATS-PCBT1090
- added C17: .1u, VupiterLinear Stage:RCL_C0402, F.Cu at (94.6, 42.7)
- added C18: .1, VupiterLinear Stage:RCL_C0402, F.Cu at (87.6, 83.3)
- added C19: .1u, VupiterLinear Stage:RCL_C0402, F.Cu at (88.9, 64.3)
- added C20: .1u, VupiterLinear Stage:RCL_C0402, F.Cu at (88.9, 27.4)
- added D1: HSMG-C170, VupiterLinear Stage:RCL_R0805, F.Cu at (44.2, 41.1)
- added R17: 1k, VupiterLinear Stage:RCL_R0805, F.Cu at (62.5, 89.4)
- added R18: R_US, VupiterLinear Stage:RCL_R0805, F.Cu at (48.8, 41.1)
- added R19: 10k, VupiterLinear Stage:RCL_R0805, F.Cu at (38.6, 46.9)
- added R20: 10k, VupiterLinear Stage:RCL_R0805, F.Cu at (41.1, 46.9)
- added R21: 10k, VupiterLinear Stage:RCL_R0805, F.Cu at (45.0, 47.5)
- added R22: 10k, VupiterLinear Stage:RCL_R0805, F.Cu at (39.2, 50.0)
- added R23: 10k, VupiterLinear Stage:RCL_R0805, F.Cu at (39.9, 57.7)
- added R24: 10k, VupiterLinear Stage:RCL_R0805, F.Cu at (39.9, 60.2)
- added R25: .5, Bourns:PWR5322WR500JE, F.Cu at (34.0, 33.0)
- added R26: .5, Bourns:PWR5322WR500JE, F.Cu at (34.0, 27.9)
- added U1: EFM8BB31F16G-C-QFN24R, Footprints:EFM8BB31F16G-C-QFN24, F.Cu at (50.0, 53.8)
- added U2: Header2Pin, Headers:Headers2Pin, F.Cu at (55.8, 48.8)
- added U3: Header5Pin, Headers:Header5Pin, F.Cu at (50.0, 45.6)
- added U4: Header5Pin, Headers:Header5Pin, F.Cu at (45.0, 53.8)
- added U5: Header5Pin, Headers:Header5Pin, F.Cu at (45.0, 64.6)
- added U6: Header4Pin, Headers:Headers4Pin, F.Cu at (53.2, 62.7)
- added U7: Header4Pin, Headers:Headers4Pin, F.Cu at (31.0, 53.8)
- added U8: Pi121U31, 2PaiSemi:Pi121U31, F.Cu at (38.6, 53.8)
- C1: footprint RCL_C0805 -> Capacitor_SMD:C_0603_1608Metric_Pad1.08x0.95mm_HandSolder
- C10, C9: value ~ -> 500p; footprint RCL_C0805 -> VupiterLinear Stage:RCL_C0805
- C11: value ~ -> 100p; footprint RCL_C0805 -> VupiterLinear Stage:RCL_C0805; moved to B.Cu
- C12: value ~ -> 100p; footprint RCL_C0805 -> VupiterLinear Stage:RCL_C0805
- C13, C14, C2, C4, C5, C6, C7, C8: footprint RCL_C0805 -> VupiterLinear Stage:RCL_C0805
- C15: value ~ -> 1u; footprint RCL_C0805 -> VupiterLinear Stage:RCL_C0805
- C16: value ~ -> .1u; footprint RCL_C0805 -> VupiterLinear Stage:RCL_C0805
- C3: footprint RCL_C0805 -> Capacitor_SMD:C_0805_2012Metric_Pad1.18x1.45mm_HandSolder
- Q1, Q2: footprint TRANSISTOR-POWER_TO220AV -> VupiterLinear Stage:TRANSISTOR-POWER_TO220AV
- R1: footprint RCL_R2512 -> VupiterLinear Stage:RCL_R2512
- R10: value ~ -> 10k; footprint RCL_R0805 -> VupiterLinear Stage:RCL_R0805
- R11, R12: footprint RCL_R0805 -> VupiterLinear Stage:RCL_R0805
- R13, R14, R16: value ~ -> 1k; footprint RCL_R0805 -> VupiterLinear Stage:RCL_R0805
- R15: value ~ -> .05; footprint RCL_R2512 -> VupiterLinear Stage:RCL_R2512
- R2: footprint RCL_R2512W -> VupiterLinear Stage:RCL_R2512W
- R3: footprint RCL_M0805 -> VupiterLinear Stage:RCL_M0805
- R4: value 6k -> 2.5k; footprint RCL_M0805 -> VupiterLinear Stage:RCL_M0805
- R5, R6: value ~ -> 50k; footprint RCL_R0805 -> VupiterLinear Stage:RCL_R0805
- R7, R8: value ~ -> 4k; footprint RCL_R0805 -> VupiterLinear Stage:RCL_R0805
- R9: value ~ -> 96k; footprint RCL_R0805 -> VupiterLinear Stage:RCL_R0805
- T1, T2: footprint TRANSISTOR_TO92 -> VupiterLinear Stage:TRANSISTOR_TO92
- U$1, U$2: footprint TEXAS_MC33063A -> VupiterLinear Stage:TEXAS_MC33063A
- U$11, U$12: footprint TEXAS_SOIC127P780X200-14N -> VupiterLinear Stage:TEXAS_SOIC127P780X200-14N
- U$13, U$15, U$29, U$4, U$9: footprint BOCHEN_3362P-1-502 -> VupiterLinear Stage:BOCHEN_3362P-1-502
- U$14, U$16, U$17, U$18, U$19, U$3, U$7: footprint ON-SEMICONDUCTOR_1N58XX -> VupiterLinear Stage:ON-SEMICONDUCTOR_1N58XX
- U$20, U$21, U$22, U$23: value MS0530 -> MS0530-1R5M; footprint COILMX_MS0530 -> VupiterLinear Stage:COILMX_MS0530
- U$27: footprint ATS_ATS-PCBT1090 -> VupiterLinear Stage:ATS_ATS-PCBT1090
- U$28: footprint JCET_LM317 -> VupiterLinear Stage:JCET_LM317
- U$31: footprint BC_BCIHP0724-4R7M -> VupiterLinear Stage:BC_BCIHP0724-4R7M
- U$6, U$8: footprint SXN_SMNR6028 -> VupiterLinear Stage:SXN_SMNR6028
- VP_0: footprint VUPITERVPAD_VPAC0 -> VupiterLinear Stage:VUPITERVPAD_VPAC0
- moved U$6 165.9 mm to (27.6, 82.8)
- moved U$4 163.8 mm to (19.3, 96.5)
- moved T2 161.7 mm to (7.62, 59.7)
- moved C4 159.1 mm to (29.0, 96.1), turned to 270 degrees
- moved C8 158.1 mm to (15.2, 59.7)
- moved U$22 158.0 mm to (22.9, 63.5), turned to 180 degrees
- moved C5 149.7 mm to (41.7, 96.0)
- moved T1 142.6 mm to (7.62, 54.6)
- moved C6 137.1 mm to (24.1, 58.7), turned to 90 degrees
- moved R3 135.3 mm to (7.62, 48.3), turned to 270 degrees
- moved C7 134.9 mm to (21.6, 58.4), turned to 90 degrees
- moved C16 128.9 mm to (61.0, 85.3), turned to 180 degrees
- moved U$27 128.0 mm to (15.2, 26.7)
- moved U$23 127.0 mm to (15.2, 63.5), turned to 180 degrees
- moved VP_0 126.4 mm to (2.54, 73.7)
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Connections:
- C1 pad 2: SGP -> ACGP
- C15 pad 2: DGP -> ACGP
- C16 pad 2: DGP -> ACGP
- C2 pad 2: SGP -> ACGP
- C3 pad 2: SGP -> ACGP
- C4 pad 2: SGP -> ACGP
- C5 pad 2: SGP -> ACGP
- C6 pad 2: PGP -> ACGP
- C7 pad 2: PGP -> ACGP
- C8 pad 2: PGP -> ACGP
- Q1 pad E: /N$19 -> Net-(Q1-PadE)
- Q2 pad E: /N$21 -> Net-(Q2-PadE)
- R15 pad 1: PGP -> /OUTP
- R3 pad 1: PGP -> ACGP
- R4 pad 1: PGP -> ACGP
- R6 pad 1: /OUTN -> /N$13
- R6 pad 2: /N$13 -> ACGP
- U$1 pad P$4: SGP -> ACGP
- U$1 pad P$5: Net-(U$1-PadP$5) -> /FB5
- U$11 pad 10: /ISET -> Net-(U$11-Pad10)
- U$11 pad 8: /N$14 -> Net-(U$11-Pad8)
- U$11 pad 9: /N$15 -> Net-(U$11-Pad9)
- U$12 pad 10: Net-(U$12-Pad10) -> /ISET
- U$12 pad 8: Net-(U$12-Pad8) -> /N$14
- U$12 pad 9: Net-(U$12-Pad9) -> /N$15
- U$2 pad P$5: Net-(U$2-PadP$5) -> /FB3
- U$27 pad P$1: PGP -> ACGP
- U$3 pad A: SGP -> ACGP
- U$4 pad P$1: Net-(U$4-PadP$1) -> ACGP
- U$8 pad P$2: SGP -> ACGP
- U$9 pad P$1: Net-(U$9-PadP$1) -> ACGP
- VP_0 pad VP: /GND -> ACGP
Routing:
- net /AD: track 0.00 -> 206.5 mm, vias 0 -> 3
- net /VCC: track 0.00 -> 140.6 mm, vias 0 -> 5
- net ACGP: track 0.00 -> 130.2 mm, vias 0 -> 24
- net /PG3: track 0.00 -> 103.8 mm, vias 0 -> 3
- net /VIN: track 0.00 -> 95.8 mm, vias 0 -> 1
- net /N$9: track 0.00 -> 88.9 mm, vias 0 -> 1
- net /OUTP: track 0.00 -> 77.2 mm, vias 0 -> 2
- net /IREAD: track 0.00 -> 75.0 mm, vias 0 -> 3
- net /VR: track 0.00 -> 72.1 mm, vias 0 -> 3
- net /ISENSE: track 0.00 -> 71.0 mm, vias 0 -> 2
- net /N$10: track 0.00 -> 67.8 mm, vias 0 -> 1
- net /5V: track 0.00 -> 65.5 mm, vias 0 -> 3
- net /ISET: track 0.00 -> 64.8 mm, vias 0 -> 4
- net /VREF: track 0.00 -> 63.5 mm, vias 0 -> 2
- net /VREAD: track 0.00 -> 62.0 mm, vias 0 -> 2
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- added copper zone on F.Cu, net ACGP
Other:
- board outline added: 100 x 100 mm
- net class ENC2B added: clearance 0.05, trace_width 0.2, via_dia 0.6, via_drill 0.4
- net class VIN added: clearance 0.2, trace_width 1.27, via_dia 1.27, via_drill 0.8
- rule trace_min: 0.2 -> 0.127
- rule via_min_drill: 0.3 -> 0.2
- rule via_min_size: 0.4 -> 0.45
- board text removed: "*** THIS IS THE DUMMY SAVE FILE *** IF YOUR ARE READING THIS MESSAGE, YOU HAVE NOT DONE A SAVE-AS IN PCBNEW TO THIS FILE NAME, WHEN IMPORTING A EAGLE PCB FILE TO A KICAD PCB FILE!"
