File: src/linear/SCH and PCB/VupiterLinear Stage.kicad_pcb (KiCad board)
At the start: 2 copper layers, 100 x 100 mm, 85 parts, among them Q1 TIP41C, Q2 TIP41C, T1 2N3904, T2 2N3904, U1 EFM8BB31F16G-C-QFN24R, U2 Header2Pin, U3 Header5Pin, U4 Header5Pin, U5 Header5Pin, U6 Header4Pin, U7 Header4Pin, U8 Pi121U31

Commit message: Add files via upload
Parts:
- added  : , VupiterLinear Stage:VUPITERVPAD_VPAC0, F.Cu at (38.7, 74.9)
- added  : , VupiterLinear Stage:VUPITERVPAD_VPAC0, F.Cu at (42.5, 74.9)
- added  : , VupiterLinear Stage:VUPITERVPAD_VPAC0, F.Cu at (36.1, 3.94)
- added  : , VupiterLinear Stage:VUPITERVPAD_VPAC0, F.Cu at (31.9, 3.94)
- added REF**: MountingHole_3.5mm, MountingHole:MountingHole_3.5mm, F.Cu at (5.71, 5.71)
- added REF**: MountingHole_3.5mm, MountingHole:MountingHole_3.5mm, F.Cu at (5.71, 92.7)
- added REF**: MountingHole_3.5mm, MountingHole:MountingHole_3.5mm, F.Cu at (92.7, 7.62)
- added VP_0: VPDEV0, VupiterLinear Stage:VUPITERVPAD_VPAC0, F.Cu at (3.05, 74.4)
- C1: value 1100p -> (none)
- C10, C9: value 500p -> (none)
- C11, C12: value 100p -> (none)
- C13, C14, C2, C4, C5, C6, C7, C8: value 10u -> (none)
- C15: value 1u -> (none)
- C16, C17, C19, C20: value .1u -> (none)
- C18, R25, R26: value .1 -> (none)
- C3: value 150p -> (none)
- D1: value HSMG-C170 -> (none)
- Q1, Q2: value TIP41C -> (none)
- R1: value .3 -> (none)
- R10, R19, R20, R21, R22, R23, R24: value 10k -> (none)
- R11, R12: value ~ -> (none)
- R13, R14, R16, R17: value 1k -> (none)
- R15: value .05 -> (none)
- R18: value R_US -> (none)
- R2: value .44 -> (none)
- R3: value 6k -> (none)
- R4: value 2.5k -> (none)
- R5, R6: value 50k -> (none)
- R7, R8: value 4k -> (none)
- R9: value 96k -> (none)
- T1, T2: value 2N3904 -> (none)
- U$1, U$2: value MC33063A-Q1 -> (none)
- U$11, U$12: value TL084HTL084H -> (none)
- U$13, U$15, U$29, U$4, U$9: value 3362P-1-502 -> (none)
- U$14, U$16, U$17, U$18, U$19, U$3, U$7: value 1N58XX -> (none)
- U$20, U$21: value MS0530-1R5M -> (none)
- U$27: value ATS-PCBT1090 -> (none)
- U$28: value LM317 -> (none)
- U$31: value BCIHP0724-4R7M -> (none)
- U$6, U$8: value SMNR6028 -> (none)
- U1: value EFM8BB31F16G-C-QFN24R -> (none)
- U2: value Header2Pin -> (none)
- U3, U4, U5: value Header5Pin -> (none)
- U6, U7: value Header4Pin -> (none)
- U8: value Pi121U31 -> (none)
- moved R15 35.0 mm to (36.8, 34.9), turned to 270 degrees
- moved U$31 8.81 mm to (12.1, 87.6)
Connections:
- U1 pad 1: /ENC2BUT -> /E2PB
- U1 pad 11: /ENC1BUT -> /E1PB
- U1 pad 7: /5CL -> /SCL
Routing:
- net OUTP: track 53.4 -> 110.1 mm, vias 3 -> 2
- net /ISENSE: track 84.2 -> 54.9 mm
- net /E1PB: track 9.70 -> 24.3 mm, vias 1 -> 4
- net ACGP: track 176.2 -> 161.9 mm, vias 23 -> 19
- net /SCL: track 0.00 -> 8.85 mm, vias 0 -> 1
- net /E2PB: track 4.84 -> 13.1 mm, vias 1 -> 2
- net /PREG: track 66.7 -> 60.8 mm
- net /VIN: track 88.3 -> 83.4 mm, vias 1 -> 0
- net /V3: track 45.6 -> 41.3 mm, vias 3 -> 2
- net /5V: track 85.8 -> 88.0 mm, vias 4 -> 3
- net /IREAD: track 53.0 -> 54.0 mm

Commit message: Add files via upload
Parts:
- removed  : , VupiterLinear Stage:VUPITERVPAD_VPAC0 (x4)
- added C21: , VupiterLinear Stage:RCL_C0805, F.Cu at (81.3, 69.8)
- added C22: , VupiterLinear Stage:RCL_C0402, F.Cu at (77.9, 61.4)
- added C23: , VupiterLinear Stage:RCL_C0402, F.Cu at (83.8, 67.9)
- added VP_0: VPDEV0, VupiterLinear Stage:VUPITERVPAD_VPAC0, F.Cu at (38.7, 74.9)
- added VP_0: VPDEV0, VupiterLinear Stage:VUPITERVPAD_VPAC0, F.Cu at (42.5, 74.9)
- added VP_0: VPDEV0, VupiterLinear Stage:VUPITERVPAD_VPAC0, F.Cu at (36.1, 3.94)
- added VP_0: VPDEV0, VupiterLinear Stage:VUPITERVPAD_VPAC0, F.Cu at (31.9, 3.94)
- C1: value (none) -> 1100p
- C10, C9: value (none) -> 500p
- C11, C12: value (none) -> 100p
- C13, C14, C2, C4, C5, C6, C7, C8: value (none) -> 10u
- C15: value (none) -> 1u
- C16, C17, C19, C20: value (none) -> .1u
- C18, R25, R26: value (none) -> .1
- C3: value (none) -> 150p
- D1: value (none) -> HSMG-C170
- Q1, Q2: value (none) -> TIP41C
- R1: value (none) -> .3
- R10, R11, R19, R20, R21, R22, R23, R24: value (none) -> 10k
- R12, R9: value (none) -> 96k
- R13, R14, R16, R17: value (none) -> 1k
- R15: value (none) -> .05
- R18: value (none) -> R_US
- R2: value (none) -> .44
- R3: value (none) -> 6k
- R4: value (none) -> 2.5k
- R5, R6: value (none) -> 50k
- R7, R8: value (none) -> 4k
- T1, T2: value (none) -> 2N3904
- U$1, U$2: value (none) -> MC33063A-Q1
- U$11, U$12: value (none) -> TL084HTL084H
- U$13, U$15, U$29, U$4, U$9: value (none) -> 3362P-1-502
- U$14, U$16, U$17, U$18, U$19, U$3, U$7: value (none) -> 1N58XX
- U$20, U$21: value (none) -> MS0530-1R5M
- U$27: value (none) -> ATS-PCBT1090
- U$28: value (none) -> LM317
- U$31: value (none) -> BCIHP0724-4R7M
- U$6, U$8: value (none) -> SMNR6028
- U1: value (none) -> EFM8BB31F16G-C-QFN24R
- U3, U4, U5: value (none) -> Header5Pin
- U6, U7: value (none) -> Header4Pin
- U8: value (none) -> Pi121U31
Connections:
- VP_0 pad VP: /VIN -> ACGP
Routing:
- net /V3: track 41.3 -> 49.6 mm
- net ACGP: track 161.9 -> 160.7 mm
