File: src/linear/SCH and PCB/VupiterLinear Stage.sch (KiCad schematic (older format))
At the start: 85 parts, among them Q1 TIP41C, Q2 TIP41C, T1 2N3904, T2 2N3904, U1 EFM8BB31F16G-C-QFN24R, U2 Header2Pin, U3 Header5Pin, U4 Header5Pin, U5 Header5Pin, U6 Header4Pin, U7 Header4Pin, U8 Pi121U31

Commit message: Add files via upload
Connections:
- net labels removed: 5CL, ENC1BUT, ENC2BUT
Changed lines of the file:
@@
 $EndComp
 Text Label 8550 3750 2    50   ~ 0
-ENC2BUT
+E2PB
 Text Label 8550 3850 2    50   ~ 0
 VREF
@@
 C2D
 Text Label 8550 4350 2    50   ~ 0
-5CL
+SCL
 Text Label 8550 4450 2    50   ~ 0
 ISET
@@
 VSET
 Text Label 8550 4750 2    50   ~ 0
-ENC1BUT
+E1PB
 Text Label 8550 4850 2    50   ~ 0
 ENC1B

Commit message: Add files via upload
Parts:
- added C21: 4.7u, VupiterLinear Stage:RCL_C0805, symbol Device:C
- added C22, C23: .1u, VupiterLinear Stage:RCL_C0402, symbol Device:C
Connections:
- wire segments 225 -> 233
Changed lines of the file:
@@
 Text GLabel 11400 8550 2    50   Input ~ 0
 OUTP
+$Comp
+L Device:C C23
+U 1 1 604791AC
+P 8000 4250
+F 0 "C23" H 8115 4296 50  0000 L CNN
+F 1 ".1u" H 8115 4205 50  0000 L CNN
+F 2 "VupiterLinear Stage:RCL_C0402" H 8038 4100 50  0001 C CNN
+F 3 "~" H 8000 4250 50  0001 C CNN
+	1    8000 4250
+	1    0    0    -1
+$EndComp
+$Comp
+L Device:C C21
+U 1 1 6047A2AB
+P 7650 4250
+F 0 "C21" H 7765 4296 50  0000 L CNN
+F 1 "4.7u" H 7765 4205 50  0000 L CNN
+F 2 "VupiterLinear Stage:RCL_C0805" H 7688 4100 50  0001 C CNN
+F 3 "~" H 7650 4250 50  0001 C CNN
+	1    7650 4250
+	1    0    0    -1
+$EndComp
+Wire Wire Line
+	8550 4050 8000 4050
+Wire Wire Line
+	7650 4050 7650 4100
+Wire Wire Line
+	8000 4100 8000 4050
+Connection ~ 8000 4050
+Wire Wire Line
+	8000 4050 7650 4050
+Wire Wire Line
+	8000 4400 8000 4450
+Wire Wire Line
+	8000 4450 7650 4450
+Wire Wire Line
+	7650 4450 7650 4400
+Text Label 7750 4450 0    50   ~ 0
+GND
+$Comp
+L Device:C C22
+U 1 1 604A8393
+P 8000 3700
+F 0 "C22" H 8115 3746 50  0000 L CNN
+F 1 ".1u" H 8115 3655 50  0000 L CNN
+F 2 "VupiterLinear Stage:RCL_C0402" H 8038 3550 50  0001 C CNN
+F 3 "~" H 8000 3700 50  0001 C CNN
+	1    8000 3700
+	1    0    0    -1
+$EndComp
+Wire Wire Line
+	8000 3850 8550 3850
+Text Label 8000 3550 0    50   ~ 0
+GND
 $EndSCHEMATC
