File: src/switched/iso/iso.sch (KiCad schematic (older format))
At the start: 68 parts, among them IC1 NCP1252ADR2G, J1 Conn_01x02, J2 Conn_01x02, J3 Conn_01x02, J4 Conn_01x02, Q1 TSD5N50MR, Q2 TSD5N50MR, T1 Transformer_1P_1S, U1 NCP5106, U2 ORPC-817C, U3 TL431LP, U4 MC34072, U5 LM317_SOT-223

Commit message: final boards and initial blinky
Parts:
- C13, C20, C21, C22, C23: Checked (none) -> yes
- IC1, T1: Checked yes -> (none)
- R10, R16, R17, R9: Link https://lcsc.com/product-detail/High-Precision-Low-TCR-SMD-Resistors_UNI-ROYAL-Uniroyal-Elec-TC0350D3902T5H_C517681.html -> https://lcsc.com/product-detail/High-Precision-Low-TCR-SMD-Resistors_UNI-ROYAL-Uniroyal-Elec-TC0350B3902T5H_C517479.html
- R13: Link https://lcsc.com/product-detail/Carbon-Film-Resistors_CCO-Chian-Chia-Elec-CF1-4W-100R-5-T52_C120031.html -> https://lcsc.com/product-detail/Carbon-Film-Resistors_CCO-Chian-Chia-Elec-CF1-6W-100R-5-T52_C119846.html
- R14, R15, R3: Link https://lcsc.com/product-detail/Carbon-Film-Resistors_CCO-C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 -> https://lcsc.com/product-detail/Carbon-Film-Resistors_Huaxi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
- R4, R5, R6, R7: Notes On PFC -> (none)
Changed lines of the file:
@@
 F 1 "1k" H 7118 4405 50  0000 L CNN
 F 2 "Resistor_THT:R_Axial_DIN0207_L6.3mm_D2.5mm_P2.54mm_Vertical" V 7090 4440 50  0001 C CNN
-F 3 "CF1/4W-1KΩ±5% T52" H 7050 4450 50  0001 C CNN
-F 4 "https://lcsc.com/product-detail/Carbon-Film-Resistors_CCO-Chian-Chia-Elec-CF1-4W-1KR-5-T52_C120055.html" H 7050 4450 50  0001 C CNN "Link"
+F 3 "CF1/6W-1KΩ±5%T52" H 7050 4450 50  0001 C CNN
+F 4 "https://lcsc.com/product-detail/Carbon-Film-Resistors_Huaxing-Mechanical-Elec-CF1-6W-1KO-5-T52_C714219.html" H 7050 4450 50  0001 C CNN "Link"
 F 5 "yes" H 7050 4450 50  0001 C CNN "Checked"
 F 6 "0.0031" H 7050 4450 50  0001 C CNN "Price"
@@
 F 1 "100" H 6968 4055 50  0000 L CNN
 F 2 "Resistor_THT:R_Axial_DIN0207_L6.3mm_D2.5mm_P2.54mm_Vertical" V 6940 4090 50  0001 C CNN
-F 3 "CF1/4W-100Ω±5% T52" H 6900 4100 50  0001 C CNN
-F 4 "https://lcsc.com/product-detail/Carbon-Film-Resistors_CCO-Chian-Chia-Elec-CF1-4W-100R-5-T52_C120031.html" H 6900 4100 50  0001 C CNN "Link"
+F 3 "CF1/6W-100Ω±5% T52" H 6900 4100 50  0001 C CNN
+F 4 "https://lcsc.com/product-detail/Carbon-Film-Resistors_CCO-Chian-Chia-Elec-CF1-6W-100R-5-T52_C119846.html" H 6900 4100 50  0001 C CNN "Link"
 F 5 "yes" H 6900 4100 50  0001 C CNN "Checked"
 F 6 "0.0052" H 6900 4100 50  0001 C CNN "Price"
@@
 F 1 "39k" H 3018 2855 50  0000 L CNN
 F 2 "Resistor_SMD:R_0603_1608Metric_Pad0.98x0.95mm_HandSolder" V 2990 2890 50  0001 C CNN
-F 3 "TC0350D3902T5H" H 2950 2900 50  0001 C CNN
-F 4 "https://lcsc.com/product-detail/High-Precision-Low-TCR-SMD-Resistors_UNI-ROYAL-Uniroyal-Elec-TC0350D3902T5H_C517681.html" H 2950 2900 50  0001 C CNN "Link"
+F 3 "TC0350B3902T5H" H 2950 2900 50  0001 C CNN
+F 4 "https://lcsc.com/product-detail/High-Precision-Low-TCR-SMD-Resistors_UNI-ROYAL-Uniroyal-Elec-TC0350B3902T5H_C517479.html" H 2950 2900 50  0001 C CNN "Link"
 F 5 "On PFC" H 2950 2900 50  0001 C CNN "Notes"
 F 6 "75" H 2950 2900 50  0001 C CNN "Working Voltage"
@@
 F 1 "39k" H 3018 1755 50  0000 L CNN
 F 2 "Resistor_SMD:R_0603_1608Metric_Pad0.98x0.95mm_HandSolder" V 2990 1790 50  0001 C CNN
-F 3 "TC0350D3902T5H" H 2950 1800 50  0001 C CNN
-F 4 "https://lcsc.com/product-detail/High-Precision-Low-TCR-SMD-Resistors_UNI-ROYAL-Uniroyal-Elec-TC0350D3902T5H_C517681.html" H 2950 1800 50  0001 C CNN "Link"
+F 3 "TC0350B3902T5H" H 2950 1800 50  0001 C CNN
+F 4 "https://lcsc.com/product-detail/High-Precision-Low-TCR-SMD-Resistors_UNI-ROYAL-Uniroyal-Elec-TC0350B3902T5H_C517479.html" H 2950 1800 50  0001 C CNN "Link"
 F 5 "On PFC" H 2950 1800 50  0001 C CNN "Notes"
 F 6 "75" H 2950 1800 50  0001 C CNN "Working Voltage"
@@
 F 1 "39k" H 9582 5995 50  0000 R CNN
 F 2 "Resistor_SMD:R_0603_1608Metric_Pad0.98x0.95mm_HandSolder" V 9690 5940 50  0001 C CNN
-F 3 "TC0350D3902T5H" H 9650 5950 50  0001 C CNN
-F 4 "https://lcsc.com/product-detail/High-Precision-Low-TCR-SMD-Resistors_UNI-ROYAL-Uniroyal-Elec-TC0350D3902T5H_C517681.html" H 9650 5950 50  0001 C CNN "Link"
+F 3 "TC0350B3902T5H" H 9650 5950 50  0001 C CNN
+F 4 "https://lcsc.com/product-detail/High-Precision-Low-TCR-SMD-Resistors_UNI-ROYAL-Uniroyal-Elec-TC0350B3902T5H_C517479.html" H 9650 5950 50  0001 C CNN "Link"
 F 5 "On PFC" H 9650 5950 50  0001 C CNN "Notes"
 F 6 "75" H 9650 5950 50  0001 C CNN "Working Voltage"
@@
 F 1 "39k" V 9514 5800 50  0000 C CNN
 F 2 "Resistor_SMD:R_0603_1608Metric_Pad0.98x0.95mm_HandSolder" V 9440 5790 50  0001 C CNN
-F 3 "TC0350D3902T5H" H 9400 5800 50  0001 C CNN
-F 4 "https://lcsc.com/product-detail/High-Precision-Low-TCR-SMD-Resistors_UNI-ROYAL-Uniroyal-Elec-TC0350D3902T5H_C517681.html" H 9400 5800 50  0001 C CNN "Link"
+F 3 "TC0350B3902T5H" H 9400 5800 50  0001 C CNN
+F 4 "https://lcsc.com/product-detail/High-Precision-Low-TCR-SMD-Resistors_UNI-ROYAL-Uniroyal-Elec-TC0350B3902T5H_C517479.html" H 9400 5800 50  0001 C CNN "Link"
 F 5 "On PFC" H 9400 5800 50  0001 C CNN "Notes"
 F 6 "75" H 9400 5800 50  0001 C CNN "Working Voltage"
@@
 F 1 "1k" H 8082 5195 50  0000 R CNN
 F 2 "Resistor_THT:R_Axial_DIN0207_L6.3mm_D2.5mm_P2.54mm_Vertical" V 8190 5140 50  0001 C CNN
-F 3 "CF1/4W-1KΩ±5% T52" H 8150 5150 50  0001 C CNN
-F 4 "https://lcsc.com/product-detail/Carbon-Film-Resistors_CCO-Chian-Chia-Elec-CF1-4W-1KR-5-T52_C120055.html" H 8150 5150 50  0001 C CNN "Link"
+F 3 "CF1/6W-1KΩ±5%T52" H 8150 5150 50  0001 C CNN
+F 4 "https://lcsc.com/product-detail/Carbon-Film-Resistors_Huaxing-Mechanical-Elec-CF1-6W-1KO-5-T52_C714219.html" H 8150 5150 50  0001 C CNN "Link"
 F 5 "yes" H 8150 5150 50  0001 C CNN "Checked"
 F 6 "0.0031" H 8150 5150 50  0001 C CNN "Price"
@@
 F 3 "WR06X100JTL" H 2400 1950 50  0001 C CNN
 F 4 "https://lcsc.com/product-detail/Chip-Resistor-Surface-Mount_Walsin-Tech-Corp-WR06X100JTL_C384297.html" H 2400 1950 50  0001 C CNN "Link"
-F 5 "On PFC" H 2400 1950 50  0001 C CNN "Notes"
+F 5 "" H 2400 1950 50  0001 C CNN "Notes"
 F 6 "75" H 2400 1950 50  0001 C CNN "Working Voltage"
 F 7 "yes" H 2400 1950 50  0001 C CNN "Checked"
@@
 F 3 "WR06X100JTL" H 2150 1450 50  0001 C CNN
 F 4 "https://lcsc.com/product-detail/Chip-Resistor-Surface-Mount_Walsin-Tech-Corp-WR06X100JTL_C384297.html" H 2150 1450 50  0001 C CNN "Link"
-F 5 "On PFC" H 2150 1450 50  0001 C CNN "Notes"
+F 5 "" H 2150 1450 50  0001 C CNN "Notes"
 F 6 "75" H 2150 1450 50  0001 C CNN "Working Voltage"
 F 7 "yes" H 2150 1450 50  0001 C CNN "Checked"
@@
 F 3 "WR06X100JTL" H 2400 1650 50  0001 C CNN
 F 4 "https://lcsc.com/product-detail/Chip-Resistor-Surface-Mount_Walsin-Tech-Corp-WR06X100JTL_C384297.html" H 2400 1650 50  0001 C CNN "Link"
-F 5 "On PFC" H 2400 1650 50  0001 C CNN "Notes"
+F 5 "" H 2400 1650 50  0001 C CNN "Notes"
 F 6 "75" H 2400 1650 50  0001 C CNN "Working Voltage"
 F 7 "yes" H 2400 1650 50  0001 C CNN "Checked"
@@
 F 3 "WR06X100JTL" H 2400 2750 50  0001 C CNN
 F 4 "https://lcsc.com/product-detail/Chip-Resistor-Surface-Mount_Walsin-Tech-Corp-WR06X100JTL_C384297.html" H 2400 2750 50  0001 C CNN "Link"
-F 5 "On PFC" H 2400 2750 50  0001 C CNN "Notes"
+F 5 "" H 2400 2750 50  0001 C CNN "Notes"
 F 6 "75" H 2400 2750 50  0001 C CNN "Working Voltage"
 F 7 "yes" H 2400 2750 50  0001 C CNN "Checked"
@@
 F 1 "1k" V 3214 6550 50  0000 C CNN
 F 2 "Resistor_THT:R_Axial_DIN0207_L6.3mm_D2.5mm_P2.54mm_Vertical" V 3140 6540 50  0001 C CNN
-F 3 "CF1/4W-1KΩ±5% T52" H 3100 6550 50  0001 C CNN
-F 4 "https://lcsc.com/product-detail/Carbon-Film-Resistors_CCO-Chian-Chia-Elec-CF1-4W-1KR-5-T52_C120055.html" H 3100 6550 50  0001 C CNN "Link"
+F 3 "CF1/6W-1KΩ±5%T52" H 3100 6550 50  0001 C CNN
+F 4 "https://lcsc.com/product-detail/Carbon-Film-Resistors_Huaxing-Mechanical-Elec-CF1-6W-1KO-5-T52_C714219.html" H 3100 6550 50  0001 C CNN "Link"
 F 5 "yes" H 3100 6550 50  0001 C CNN "Checked"
 F 6 "0.0031" H 3100 6550 50  0001 C CNN "Price"
@@
 F 2 "custom:CSV-E25-13-7-1S-6P-C" H 3900 2300 50  0001 C CNN
 F 3 "custom" H 3900 2300 50  0001 C CNN
-F 4 "yes" H 3900 2300 50  0001 C CNN "Checked"
+F 4 "" H 3900 2300 50  0001 C CNN "Checked"
 F 5 "1.337" H 3900 2300 50  0001 C CNN "Price"
 	1    3900 2300
@@
 F 2 "Package_SO:SOIC-8_3.9x4.9mm_P1.27mm" H 4550 6400 50  0001 L CNN
 F 3 "https://www.onsemi.com/pub/Collateral/NCP1252-D.PDF" H 4550 6300 50  0001 L CNN
-F 4 "yes" H 3700 6300 50  0001 C CNN "Checked"
+F 4 "" H 3700 6300 50  0001 C CNN "Checked"
 F 5 "0.5338" H 3700 6300 50  0001 C CNN "Price"
 	1    3700 6300
@@
 F 3 "C1206X5R106K500NT" H 5600 2300 50  0001 C CNN
 F 4 "https://lcsc.com/product-detail/Multilayer-Ceramic-Capacitors-MLCC-SMD-SMT_SANYEAR-C1206X5R106K500NT_C466808.html" H 5600 2300 50  0001 C CNN "Link"
-F 5 "" H 5600 2300 50  0001 C CNN "Checked"
+F 5 "yes" H 5600 2300 50  0001 C CNN "Checked"
 F 6 "" H 5600 2300 50  0001 C CNN "Working Voltage"
 F 7 "" H 5600 2300 50  0001 C CNN "Price"
@@
 F 3 "C1206X5R106K500NT" H 5950 2300 50  0001 C CNN
 F 4 "https://lcsc.com/product-detail/Multilayer-Ceramic-Capacitors-MLCC-SMD-SMT_SANYEAR-C1206X5R106K500NT_C466808.html" H 5950 2300 50  0001 C CNN "Link"
-F 5 "" H 5950 2300 50  0001 C CNN "Checked"
+F 5 "yes" H 5950 2300 50  0001 C CNN "Checked"
 F 6 "" H 5950 2300 50  0001 C CNN "Working Voltage"
 F 7 "" H 5950 2300 50  0001 C CNN "Price"
@@
 F 3 "C1206X5R106K500NT" H 6350 2300 50  0001 C CNN
 F 4 "https://lcsc.com/product-detail/Multilayer-Ceramic-Capacitors-MLCC-SMD-SMT_SANYEAR-C1206X5R106K500NT_C466808.html" H 6350 2300 50  0001 C CNN "Link"
-F 5 "" H 6350 2300 50  0001 C CNN "Checked"
+F 5 "yes" H 6350 2300 50  0001 C CNN "Checked"
 F 6 "" H 6350 2300 50  0001 C CNN "Working Voltage"
 F 7 "" H 6350 2300 50  0001 C CNN "Price"
@@
 F 3 "C1206X5R106K500NT" H 6700 2300 50  0001 C CNN
 F 4 "https://lcsc.com/product-detail/Multilayer-Ceramic-Capacitors-MLCC-SMD-SMT_SANYEAR-C1206X5R106K500NT_C466808.html" H 6700 2300 50  0001 C CNN "Link"
-F 5 "" H 6700 2300 50  0001 C CNN "Checked"
+F 5 "yes" H 6700 2300 50  0001 C CNN "Checked"
 F 6 "" H 6700 2300 50  0001 C CNN "Working Voltage"
 F 7 "" H 6700 2300 50  0001 C CNN "Price"
@@
 F 3 "C1206X5R106K500NT" H 7050 2300 50  0001 C CNN
 F 4 "https://lcsc.com/product-detail/Multilayer-Ceramic-Capacitors-MLCC-SMD-SMT_SANYEAR-C1206X5R106K500NT_C466808.html" H 7050 2300 50  0001 C CNN "Link"
-F 5 "" H 7050 2300 50  0001 C CNN "Checked"
+F 5 "yes" H 7050 2300 50  0001 C CNN "Checked"
 F 6 "" H 7050 2300 50  0001 C CNN "Working Voltage"
 F 7 "" H 7050 2300 50  0001 C CNN "Price"
